File: Audio/LME49810/LME49810.sch (KiCad schematic (older format))
At the start: 40 parts, among them P1 CONN_01X01, P10 CONN_01X01, P11 CONN_01X01, P2 CONN_01X01, P3 CONN_01X01, P4 CONN_01X01, P5 CONN_01X01, P6 CONN_01X01, P7 CONN_01X01, P8 CONN_01X01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

Commit message: Further revision
More fixes
Parts:
- C10, C2, C4, C6: footprint Capacitors_ThroughHole:C_Disc_D6_P5 -> Capacitors_ThroughHole:C_Rect_L13_W6_H12_P10
Connections:
- net labels removed: GND2
- wire segments 129 -> 127
Changed lines of the file:
@@
 EESchema Schematic File Version 2
+LIBS:74xgxx
+LIBS:74xx
+LIBS:ac-dc
+LIBS:actel
+LIBS:adc-dac
+LIBS:Altera
+LIBS:analog_devices
+LIBS:analog_switches
+LIBS:atmel
+LIBS:audio
+LIBS:brooktre
+LIBS:cmos_ieee
+LIBS:cmos4000
+LIBS:conn
+LIBS:contrib
+LIBS:cypress
+LIBS:dc-dc
+LIBS:device
+LIBS:digital-audio
+LIBS:diode
+LIBS:display
+LIBS:dsp
+LIBS:elec-unifil
+LIBS:ESD_Protection
+LIBS:ftdi
+LIBS:gennum
+LIBS:graphic
+LIBS:hc11
+LIBS:intel
+LIBS:interface
+LIBS:ir
+LIBS:Lattice
+LIBS:linear
+LIBS:logo
+LIBS:maxim
+LIBS:memory
+LIBS:microchip
+LIBS:microchip_dspic33dsc
+LIBS:microchip_pic10mcu
+LIBS:microchip_pic12mcu
+LIBS:microchip_pic16mcu
+LIBS:microchip_pic18mcu
+LIBS:microchip_pic32mcu
+LIBS:microcontrollers
+LIBS:motor_drivers
+LIBS:motorola
+LIBS:msp430
+LIBS:nordicsemi
+LIBS:nxp_armmcu
+LIBS:onsemi
+LIBS:opto
+LIBS:Oscillators
+LIBS:philips
+LIBS:power
+LIBS:Power_Management
+LIBS:powerint
+LIBS:pspice
+LIBS:references
+LIBS:regul
+LIBS:relays
+LIBS:rfcom
+LIBS:sensors
+LIBS:silabs
+LIBS:siliconi
+LIBS:stm8
+LIBS:stm32
+LIBS:supertex
+LIBS:switches
+LIBS:texas
+LIBS:transf
+LIBS:transistors
+LIBS:ttl_ieee
+LIBS:valves
+LIBS:video
+LIBS:Xicor
+LIBS:xilinx
+LIBS:Zilog
 LIBS:LME49810-rescue
-LIBS:power
-LIBS:device
-LIBS:transistors
-LIBS:conn
-LIBS:linear
-LIBS:regul
-LIBS:74xx
-LIBS:cmos4000
-LIBS:adc-dac
-LIBS:memory
-LIBS:xilinx
-LIBS:microcontrollers
-LIBS:dsp
-LIBS:microchip
-LIBS:analog_switches
-LIBS:motorola
-LIBS:texas
-LIBS:intel
-LIBS:audio
-LIBS:interface
-LIBS:digital-audio
-LIBS:philips
-LIBS:display
-LIBS:cypress
-LIBS:siliconi
-LIBS:opto
-LIBS:atmel
-LIBS:contrib
-LIBS:valves
 LIBS:lme49810
 LIBS:LME49810-cache
@@
 F 0 "C4" H 2375 1600 50  0000 L CNN
 F 1 "0.1u" H 2375 1400 50  0000 L CNN
-F 2 "Capacitors_ThroughHole:C_Disc_D6_P5" H 2388 1350 30  0001 C CNN
+F 2 "Capacitors_ThroughHole:C_Rect_L13_W6_H12_P10" H 2388 1350 30  0001 C CNN
 F 3 "" H 2350 1500 60  0000 C CNN
 	1    2350 1500
@@
 F 0 "C10" H 2575 4350 50  0000 L CNN
 F 1 "0.1u" H 2575 4150 50  0000 L CNN
-F 2 "Capacitors_ThroughHole:C_Disc_D6_P5" H 2588 4100 30  0001 C CNN
+F 2 "Capacitors_ThroughHole:C_Rect_L13_W6_H12_P10" H 2588 4100 30  0001 C CNN
 F 3 "" H 2550 4250 60  0000 C CNN
 	1    2550 4250
@@
 $EndComp
 $Comp
-L GND1 #PWR2
+L GND1 #PWR01
 U 1 1 5645FC55
 P 1800 3150
-F 0 "#PWR2" H 1800 2900 50  0001 C CNN
+F 0 "#PWR01" H 1800 2900 50  0001 C CNN
 F 1 "GND1" H 1800 3000 50  0000 C CNN
 F 2 "" H 1800 3150 60  0000 C CNN
@@
 Text GLabel 4300 2250 2    60   Output ~ 0
 SourceLH
-$Comp
-L PWR_FLAG #FLG6
-U 1 1 5645DA06
-P 5050 6000
-F 0 "#FLG6" H 5050 6095 50  0001 C CNN
-F 1 "PWR_FLAG" H 5050 6180 50  0000 C CNN
-F 2 "" H 5050 6000 60  0000 C CNN
-F 3 "" H 5050 6000 60  0000 C CNN
-	1    5050 6000
-	-1   0    0    -1
-$EndComp
 Text GLabel 6800 6000 1    60   Output ~ 0
 +5V
 $Comp
-L +5V #PWR10
+L +5V #PWR02
 U 1 1 564676E3
 P 6300 6000
-F 0 "#PWR10" H 6300 5850 50  0001 C CNN
+F 0 "#PWR02" H 6300 5850 50  0001 C CNN
 F 1 "+5V" H 6300 6140 50  0000 C CNN
 F 2 "" H 6300 6000 60  0000 C CNN
@@
 $EndComp
 $Comp
-L PWR_FLAG #FLG7
+L PWR_FLAG #FLG03
 U 1 1 56468C02
 P 6300 6100
-F 0 "#FLG7" H 6300 6195 50  0001 C CNN
+F 0 "#FLG03" H 6300 6195 50  0001 C CNN
 F 1 "PWR_FLAG" H 6300 6280 50  0000 C CNN
 F 2 "" H 6300 6100 60  0000 C CNN
@@
 -VeeL1
 $Comp
-L PWR_FLAG #FLG1
+L PWR_FLAG #FLG04
 U 1 1 5649D634
 P 1650 5950
-F 0 "#FLG1" H 1650 6045 50  0001 C CNN
+F 0 "#FLG04" H 1650 6045 50  0001 C CNN
 F 1 "PWR_FLAG" H 1650 6130 50  0000 C CNN
 F 2 "" H 1650 5950 60  0000 C CNN
@@
 $EndComp
 $Comp
-L PWR_FLAG #FLG2
+L PWR_FLAG #FLG05
 U 1 1 5649D63B
 P 2150 5950
-F 0 "#FLG2" H 2150 6045 50  0001 C CNN
+F 0 "#FLG05" H 2150 6045 50  0001 C CNN
 F 1 "PWR_FLAG" H 2150 6130 50  0000 C CNN
 F 2 "" H 2150 5950 60  0000 C CNN
@@
 	3850 3100 3700 3100
 Wire Wire Line
-	5050 6100 5050 6000
-Wire Wire Line
 	6300 6000 6300 6100
 Wire Wire Line
@@
 Wire Wire Line
 	5500 3200 5500 4150
-Connection ~ 1800 4200
-Connection ~ 5050 6050
 Wire Wire Line
 	5500 2800 5500 2900
@@
 Connection ~ 2000 6050
 $Comp
-L VCC1 #PWR6
+L VCC1 #PWR06
 U 1 1 56494154
 P 1800 6000
-F 0 "#PWR6" H 1800 5850 50  0001 C CNN
+F 0 "#PWR06" H 1800 5850 50  0001 C CNN
 F 1 "VCC1" H 1800 6150 50  0000 C CNN
 F 2 "" H 1800 6000 60  0000 C CNN
@@
 $EndComp
 $Comp
-L VEE1 #PWR7
+L VEE1 #PWR07
 U 1 1 564941D4
 P 2000 6000
-F 0 "#PWR7" H 2000 5850 50  0001 C CNN
+F 0 "#PWR07" H 2000 5850 50  0001 C CNN
 F 1 "VEE1" H 2000 6150 50  0000 C CNN
 F 2 "" H 2000 6000 60  0000 C CNN
@@
 $EndComp
 $Comp
-L VCC2 #PWR8
+L VCC2 #PWR08
 U 1 1 56494254
 P 3200 6000
-F 0 "#PWR8" H 3200 5850 50  0001 C CNN
+F 0 "#PWR08" H 3200 5850 50  0001 C CNN
 F 1 "VCC2" H 3200 6150 50  0000 C CNN
 F 2 "" H 3200 6000 60  0000 C CNN
@@
 $EndComp
 $Comp
-L VEE2 #PWR9
+L VEE2 #PWR09
 U 1 1 564942D4
 P 3400 6000
-F 0 "#PWR9" H 3400 5850 50  0001 C CNN
+F 0 "#PWR09" H 3400 5850 50  0001 C CNN
 F 1 "VEE2" H 3400 6150 50  0000 C CNN
 F 2 "" H 3400 6000 60  0000 C CNN
@@
 -VeeL2
 $Comp
-L PWR_FLAG #FLG3
+L PWR_FLAG #FLG010
 U 1 1 564A7742
 P 3050 5950
-F 0 "#FLG3" H 3050 6045 50  0001 C CNN
+F 0 "#FLG010" H 3050 6045 50  0001 C CNN
 F 1 "PWR_FLAG" H 3050 6130 50  0000 C CNN
 F 2 "" H 3050 5950 60  0000 C CNN
@@
 $EndComp
 $Comp
-L PWR_FLAG #FLG4
+L PWR_FLAG #FLG011
 U 1 1 564A7748
 P 3550 5950
-F 0 "#FLG4" H 3550 6045 50  0001 C CNN
+F 0 "#FLG011" H 3550 6045 50  0001 C CNN
 F 1 "PWR_FLAG" H 3550 6130 50  0000 C CNN
 F 2 "" H 3550 5950 60  0000 C CNN
@@
 F 0 "C2" H 9075 1500 50  0000 L CNN
 F 1 "0.1u" H 9075 1300 50  0000 L CNN
-F 2 "Capacitors_ThroughHole:C_Disc_D6_P5" H 9088 1250 30  0001 C CNN
+F 2 "Capacitors_ThroughHole:C_Rect_L13_W6_H12_P10" H 9088 1250 30  0001 C CNN
 F 3 "" H 9050 1400 60  0000 C CNN
 	1    9050 1400
@@
 F 0 "C6" H 9075 2800 50  0000 L CNN
 F 1 "0.1u" H 9075 2600 50  0000 L CNN
-F 2 "Capacitors_ThroughHole:C_Disc_D6_P5" H 9088 2550 30  0001 C CNN
+F 2 "Capacitors_ThroughHole:C_Rect_L13_W6_H12_P10" H 9088 2550 30  0001 C CNN
 F 3 "" H 9050 2700 60  0000 C CNN
 	1    9050 2700
@@
 $EndComp
 $Comp
-L GND2 #PWR12
-U 1 1 564DD122
-P 5050 6100
-F 0 "#PWR12" H 5050 5850 50  0001 C CNN
-F 1 "GND2" H 5050 5950 50  0000 C CNN
-F 2 "" H 5050 6100 60  0000 C CNN
-F 3 "" H 5050 6100 60  0000 C CNN
-	1    5050 6100
-	-1   0    0    -1
-$EndComp
-$Comp
 L R-RESCUE-LME49810 R1
 U 1 1 564BFF29
@@
 	5300 6000 5300 6050
 Wire Wire Line
-	5050 6050 5800 6050
-$Comp
-L PWR_FLAG #FLG5
+	4250 6050 5800 6050
+$Comp
+L PWR_FLAG #FLG012
 U 1 1 564C200E
 P 4750 6000
-F 0 "#FLG5" H 4750 6095 50  0001 C CNN
+F 0 "#FLG012" H 4750 6095 50  0001 C CNN
 F 1 "PWR_FLAG" H 4750 6180 50  0000 C CNN
 F 2 "" H 4750 6000 60  0000 C CNN
@@
 Wire Wire Line
 	4500 6000 4500 6050
-Wire Wire Line
-	4250 6050 4750 6050
 $Comp
 L CONN_01X01 P9
@@
 	5800 6050 5800 6000
 Connection ~ 5550 6050
-Text GLabel 5800 6000 1    60   Output ~ 0
-GND2
 Text GLabel 4250 6000 1    60   Output ~ 0
 GND1
@@
 	2150 1850 2150 1750
 Connection ~ 2350 1750
-Text GLabel 8750 1700 3    60   Input ~ 0
-GND2
-Text GLabel 9050 1700 3    60   Input ~ 0
-GND2
-Text GLabel 8750 3000 3    60   Input ~ 0
-GND2
-Text GLabel 9050 3000 3    60   Input ~ 0
-GND2
 Text Label 7100 1600 0    60   ~ 0
 Emit-NPN
@@
 Emit-PNP
 $Comp
-L GND1 #PWR3
+L GND1 #PWR013
 U 1 1 564C1A71
 P 950 3950
-F 0 "#PWR3" H 950 3700 50  0001 C CNN
+F 0 "#PWR013" H 950 3700 50  0001 C CNN
 F 1 "GND1" H 950 3800 50  0000 C CNN
 F 2 "" H 950 3950 60  0000 C CNN
@@
 $EndComp
 $Comp
-L GND1 #PWR4
-U 1 1 564C1AF1
-P 3400 3950
-F 0 "#PWR4" H 3400 3700 50  0001 C CNN
-F 1 "GND1" H 3400 3800 50  0000 C CNN
-F 2 "" H 3400 3950 60  0000 C CNN
-F 3 "" H 3400 3950 60  0000 C CNN
-	1    3400 3950
-	1    0    0    -1
-$EndComp
-$Comp
-L GND1 #PWR1
+L GND1 #PWR014
 U 1 1 564C1B71
 P 2150 1850
-F 0 "#PWR1" H 2150 1600 50  0001 C CNN
+F 0 "#PWR014" H 2150 1600 50  0001 C CNN
 F 1 "GND1" H 2150 1700 50  0000 C CNN
 F 2 "" H 2150 1850 60  0000 C CNN
@@
 $EndComp
 $Comp
-L GND1 #PWR5
+L GND1 #PWR015
 U 1 1 564C1C18
 P 2150 4600
-F 0 "#PWR5" H 2150 4350 50  0001 C CNN
+F 0 "#PWR015" H 2150 4350 50  0001 C CNN
 F 1 "GND1" H 2150 4450 50  0000 C CNN
 F 2 "" H 2150 4600 60  0000 C CNN
@@
 	6100 2000 6100 2150
 $Comp
-L GND1 #PWR11
+L GND1 #PWR016
 U 1 1 564C201C
 P 4750 6100
-F 0 "#PWR11" H 4750 5850 50  0001 C CNN
+F 0 "#PWR016" H 4750 5850 50  0001 C CNN
 F 1 "GND1" H 4750 5950 50  0000 C CNN
 F 2 "" H 4750 6100 60  0000 C CNN
@@
 Wire Wire Line
 	10000 1950 10200 1950
+Text GLabel 3400 3950 3    60   Input ~ 0
+GND1
+Text GLabel 8750 1700 3    60   Input ~ 0
+GND1
+Text GLabel 9050 1700 3    60   Input ~ 0
+GND1
+Text GLabel 8750 3000 3    60   Input ~ 0
+GND1
+Text GLabel 9050 3000 3    60   Input ~ 0
+GND1
 $EndSCHEMATC

Commit message: Improvements
PCB revised.
Parts:
- removed P1, P10, P11, P2, P3, P4, P5, P6, P7, P8, P9: CONN_01X01, LME49810:Soldering_pad, symbol CONN_01X01
- added R14, R15: 10, Resistors_ThroughHole:Resistor_Horizontal_RM10mm, symbol R-RESCUE-LME49810
- C1, C5: value 4700u -> 820u,100V; footprint Capacitors_ThroughHole:C_Radial_D18_L36_P7.5 -> Capacitors_ThroughHole:C_Radial_D16_L31.5_P7.5
- C3, C9: value 470u -> 820u,100V
Connections:
- wire segments 127 -> 118
- no-connect marks 2 -> 3
Other:
- moved on the sheet: R1, R2, R4, R5, R6

Commit message: Fixes
More fixes done
Parts:
- added C11: 470u, Capacitors_ThroughHole:C_Radial_D8_L11.5_P3.5, symbol CP1-RESCUE-LME49810
- added P1, P2, P3, P4, P5: CONN_01X01, Connect:PINTST, symbol CONN_01X01
- C10, C2, C4, C6: footprint Capacitors_ThroughHole:C_Rect_L13_W6_H12_P10 -> Capacitors_ThroughHole:C_Rect_L18_W6_H12_P15
- D1: footprint LEDs:LED-3MM -> LEDs:LED-5MM
- Q1, Q2: footprint Transistors_TO-247:TO-247_Vertical_Neutral123 -> TO_SOT_Packages_THT:TO-247_Vertical_Neutral123_MountedFromLS
- Q3: footprint Transistors_TO-220:TO-220_Neutral123_Vertical -> TO_SOT_Packages_THT:TO-220_Neutral123_Vertical_LargePads
- R11, R7: value 240 -> 470
- R12: value 6.8k -> 7.5k
- R13, R14, R15, R6: footprint Resistors_ThroughHole:Resistor_Horizontal_RM10mm -> Resistors_ThroughHole:Resistor_Horizontal_RM15mm
- R8: value 6.8k -> 7.5k; footprint Resistors_ThroughHole:Resistor_Horizontal_RM10mm -> Resistors_ThroughHole:Resistor_Horizontal_RM15mm
- R9: value 360 -> 330
- RV1: value 200 -> 500
Connections:
- net Emit-NPN: now also Q1.3 (E), R2.2, P1.1 (P1)
- net Emit-PNP: now also Q2.3 (E), R4.1, P2.1 (P1)
- net GND1: now also C11.2
- net Vee: now reaches C10.2, C9.2, R14.2, U1.10 (-Vee)
- net Vcc: now reaches C3.1, C4.1, R15.2, U1.15 (+Vcc)
- net at D1.1 (A): now also R13.2, P5.1 (P1); no longer R13.1
- net IN-: now reaches C8.1, R11.1
- net +5V: no longer names the net of R6.2
- net +5V: now also P3.1 (P1); no longer R13.2
- net InputLH renamed IN+
- net IN+: now also C11.1
- new net: P4.1 (P1), R13.1
- no-connect marks 3 -> 2
Other:
- moved on the sheet: C8
