File: Audio/LME49810/LME49810.kicad_pcb (KiCad board)
At the start: 2 copper layers, 81.3 x 94 mm, 40 parts, among them P1 CONN_01X01, P10 CONN_01X01, P11 CONN_01X01, P2 CONN_01X01, P3 CONN_01X01, P4 CONN_01X01, P5 CONN_01X01, P6 CONN_01X01, P7 CONN_01X01, P8 CONN_01X01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

Commit message: Further revision
More fixes
Parts:
- removed P11, P7, P8, P9: CONN_01X01, LME49810:Soldering_pad
- C10, C2, C4, C6: footprint Capacitors_ThroughHole:C_Disc_D6_P5 -> Capacitors_ThroughHole:C_Rect_L18_W6_H12_P15
- R12, R8: footprint Resistors_ThroughHole:Resistor_Horizontal_RM10mm -> Resistors_ThroughHole:Resistor_Horizontal_RM15mm
- moved C8 20.7 mm to (67.9, 45.1), turned to 90 degrees
- moved R8 19.9 mm to (91.4, 68.6)
- moved C10 17.7 mm to (98.8, 73.7)
- moved P1 17.1 mm to (52.1, 71.8)
- moved P6 16.2 mm to (41.9, 55.9)
- moved P5 16.2 mm to (41.9, 88.9)
- moved R10 15.9 mm to (31.1, 74.9), turned to 90 degrees
- moved C6 15.2 mm to (62.2, 55.9)
- moved R6 15.1 mm to (78.1, 54.6)
- moved R7 13.2 mm to (81.6, 61.3), turned to 270 degrees
- moved R12 12.0 mm to (59.7, 66.0), turned to 180 degrees
- moved P3 11.4 mm to (92.7, 91.4)
- moved P4 10.9 mm to (92.7, 62.2)
- moved RV1 10.8 mm to (43.2, 71.1), turned to 180 degrees
- moved R13 10.3 mm to (73.7, 49.5)
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Connections:
- C1 pad 2: GND2 -> GND1
- C2 pad 2: GND2 -> GND1
- C5 pad 1: GND2 -> GND1
- C6 pad 1: GND2 -> GND1
Routing:
- net GND1: track 77.0 -> 15.9 mm
- net GND2: track 37.6 -> 0.00 mm
- net -VeeL2: track 37.9 -> 63.7 mm
- net +VccL2: track 37.7 -> 63.1 mm
- net -VeeL1: track 22.8 -> 41.1 mm
- net OUTLH: track 23.8 -> 41.4 mm, vias 0 -> 1
- net +VccL1: track 25.2 -> 39.8 mm
- net CLH: track 37.7 -> 52.2 mm
- net Net-(R7-Pad2): track 22.3 -> 8.67 mm
- net Net-(Q1-Pad1): track 5.29 -> 18.9 mm
- net Net-(R6-Pad1): track 17.9 -> 5.52 mm
- net +5V: track 19.1 -> 6.92 mm
- net Net-(R9-Pad2): track 18.6 -> 9.68 mm
- net ELH: track 36.2 -> 43.9 mm
- net Net-(R11-Pad2): track 14.2 -> 6.88 mm
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- added copper zone on B.Cu, net GND1

Commit message: Improvements
PCB revised.
Parts:
- removed P1, P10, P2, P3, P4, P5, P6: CONN_01X01, LME49810:Soldering_pad
- added R14: 10, Resistors_ThroughHole:Resistor_Horizontal_RM10mm, F.Cu at (87.6, 59.7)
- added R15: 10, Resistors_ThroughHole:Resistor_Horizontal_RM10mm, F.Cu at (82.5, 88.9)
- C1, C5: value 4700u -> 820u,100V; footprint Capacitors_ThroughHole:C_Radial_D18_L36_P7.5 -> Capacitors_ThroughHole:C_Radial_D16_L31.5_P7.5
- C3, C9: value 470u -> 820u,100V
- R12: footprint Resistors_ThroughHole:Resistor_Horizontal_RM15mm -> Resistors_ThroughHole:Resistor_Horizontal_RM10mm
- moved C9 10.2 mm to (100.3, 47.0)
- moved R13 3.42 mm to (74.9, 52.7)
- moved R12 2.62 mm to (57.1, 65.4)
- moved R11 2.01 mm to (67.9, 60.3)
- moved R6 1.91 mm to (78.1, 52.7)
- moved D1 1.42 mm to (72.4, 57.8)
- moved C3 1.27 mm to (92.7, 97.8)
- moved R8 0.64 mm to (92.1, 68.6)
- moved C7 0.51 mm to (68.6, 73.6)
- moved R7 0.34 mm to (81.9, 61.3)
Connections:
- net +VccL1 renamed Net-(C3-Pad1)
- net -VeeL1 renamed Net-(C10-Pad2)
- net /Emit-NPN renamed Net-(Q1-Pad3)
- net /Emit-PNP renamed Net-(Q2-Pad3)
- U1 pad 7: (no net) -> Net-(U1-Pad7)
- U1 pad 9: (no net) -> Net-(U1-Pad9)
Routing:
- net /InputLH: track 7.96 -> 0.00 mm
- net Net-(R11-Pad2): track 6.88 -> 13.5 mm
- net +5V: track 6.92 -> 3.17 mm
- net ELH: track 43.9 -> 46.8 mm
- net Net-(R7-Pad2): track 8.67 -> 10.9 mm
- net Net-(R6-Pad1): track 5.52 -> 7.42 mm
- net CLH: track 52.2 -> 54.1 mm
- net Net-(C8-Pad1): track 11.6 -> 10.2 mm
- net Net-(C3-Pad1): track 39.8 -> 38.5 mm
- net Net-(D1-Pad1): track 2.54 -> 3.18 mm

Commit message: Fixes
More fixes done
Parts:
- added C11: 470u, Capacitors_ThroughHole:C_Radial_D8_L11.5_P3.5, F.Cu at (82.5, 43.8)
- added P1: CONN_01X01, Connect:PINTST, F.Cu at (50.8, 77.5)
- added P2: CONN_01X01, Connect:PINTST, F.Cu at (50.8, 44.5)
- added P3: CONN_01X01, Connect:PINTST, F.Cu at (79.4, 29.2)
- added P4: CONN_01X01, Connect:PINTST, F.Cu at (71.8, 29.2)
- added P5: CONN_01X01, Connect:PINTST, F.Cu at (73.7, 47.0)
- D1: footprint LEDs:LED-3MM -> LEDs:LED-5MM
- Q1, Q2: footprint Transistors_TO-247:TO-247_Vertical_Neutral123 -> TO_SOT_Packages_THT:TO-247_Vertical_Neutral123_MountedFromLS
- Q3: footprint Transistors_TO-220:TO-220_Neutral123_Vertical -> TO_SOT_Packages_THT:TO-220_Neutral123_Vertical_LargePads
- R11, R7: value 240 -> 470
- R12, R8: value 6.8k -> 7.5k
- R13, R14, R15, R6: footprint Resistors_ThroughHole:Resistor_Horizontal_RM10mm -> Resistors_ThroughHole:Resistor_Horizontal_RM15mm
- R9: value 360 -> 330
- RV1: value 200 -> 500
- moved R6 16.0 mm to (76.8, 36.7)
- moved R13 16.0 mm to (74.3, 36.7), turned to 270 degrees
- moved R15 15.3 mm to (97.8, 87.6), turned to 180 degrees
- moved R1 11.4 mm to (62.2, 94.6)
- moved R14 10.6 mm to (97.8, 56.5), turned to 180 degrees
- moved R3 8.91 mm to (66.7, 78.1), turned to 135 degrees
- moved D1 8.35 mm to (73.7, 49.5)
- moved C5 7.73 mm to (47.0, 30.5), turned to 270 degrees
- moved RV1 7.73 mm to (50.8, 72.4), turned to 90 degrees
- moved R5 7.18 mm to (55.9, 67.3)
- moved C1 6.35 mm to (47.0, 106.7), turned to 270 degrees
- moved R9 6.02 mm to (41.9, 72.4), turned to 270 degrees
- moved R8 5.14 mm to (92.8, 63.5)
- moved C10 5.08 mm to (98.8, 68.6)
- moved R12 4.26 mm to (61.0, 63.5)
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Connections:
- net Net-(C10-Pad2) renamed /Vee
- net Net-(C3-Pad1) renamed /Vcc
- net Net-(C8-Pad1) renamed /IN-
- net Net-(Q1-Pad3) renamed /Emit-NPN
- net Net-(Q2-Pad3) renamed /Emit-PNP
- R13 pad 1: Net-(D1-Pad1) -> Net-(P4-Pad1)
- R13 pad 2: +5V -> Net-(D1-Pad1)
- R14 pad 1: -VeeL1 -> (no net)
- R15 pad 1: +VccL1 -> (no net)
- R6 pad 2: +5V -> Net-(P3-Pad1)
- R7 pad 1: /InputLH -> /IN+
- U1 pad 7: Net-(U1-Pad7) -> (no net)
- U1 pad 9: Net-(U1-Pad9) -> (no net)
Routing:
- net OUTLH: track 41.4 -> 70.5 mm
- net -VeeL2: track 63.7 -> 45.1 mm
- net +VccL2: track 63.1 -> 44.8 mm
- net Net-(R6-Pad1): track 7.42 -> 21.0 mm
- net SourceLH: track 33.8 -> 21.8 mm
- net /Emit-PNP: track 5.40 -> 15.1 mm
- net /Emit-NPN: track 5.40 -> 15.1 mm
- net /IN+: track 0.00 -> 9.53 mm
- net SinkLH: track 28.8 -> 19.7 mm
- net Net-(D1-Pad2): track 4.16 -> 11.4 mm
- net Net-(Q2-Pad1): track 10.7 -> 15.1 mm
- net CLH: track 54.1 -> 50.1 mm
- net Net-(D1-Pad1): track 3.18 -> 6.85 mm
- net Net-(R11-Pad2): track 13.5 -> 9.94 mm
- net Net-(C7-Pad2): track 9.77 -> 6.49 mm
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Other:
- board size 81.3 x 94 mm -> 86.4 x 99.1 mm
- net class Default: trace_width 1 -> 1.5; via_dia 2 -> 1.5; via_drill 1 -> 0.75
- net class Thick: trace_width 3 -> 4
- board text added: "GND"
- board text added: "IN+"
- board text added: "IN-"
- board text added: "MUTE"
- board text added: "OUT"
- board text added: "PEAK"
- board text added: "TDU Audio Technology Research Club"
- board text added: "Vcc(1)"
- board text added: "Vcc(2)"
- board text added: "Vee(1)"
- board text added: "Vee(2)"
- board text added: "○"
- board text removed: "X"

Commit message: Fixes on component conflict
LME49810 PCB revised
Routing:
- net Net-(R11-Pad2): track 9.94 -> 10.5 mm
Other:
- board text added: "Audio Technology Research Club at Tokyo Denki University"
- board text added: "LME49810 Power Amplifier PCB Designed by T.Hashizume Dec.2015"
- board text removed: "TDU Audio Technology Research Club"
Changed lines of the file:
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@@
     (links 56)
     (no_connects 0)
-    (area 14.860001 17.47 111.860001 121.970001)
+    (area 14.860001 17.47 112.010001 122.170001)
     (thickness 1.6)
-    (drawings 24)
-    (tracks 133)
+    (drawings 25)
+    (tracks 134)
     (zones 0)
     (modules 37)
@@
     (trace_min 0.1)
     (segment_width 0.2)
-    (edge_width 0.1)
+    (edge_width 0.5)
     (via_size 1.5)
     (via_drill 0.75)
@@
     )
   )
+  (gr_text "LME49810 Power Amplifier PCB\nDesigned by T.Hashizume\nDec.2015" (at 82.55 115.57) (layer B.Cu)
+    (effects (font (size 1.5 1.5) (thickness 0.3)) (justify mirror))
+  )
   (gr_line (start 25.4 72.39) (end 111.76 72.39) (angle 90) (layer Dwgs.User) (width 0.2))
   (gr_text ○ (at 30.48 83.82) (layer B.Cu)
@@
     (effects (font (size 1.5 1.5) (thickness 0.3)) (justify mirror))
   )
-  (gr_line (start 25.4 121.92) (end 25.4 22.86) (angle 90) (layer Edge.Cuts) (width 0.1))
-  (gr_line (start 111.76 121.92) (end 25.4 121.92) (angle 90) (layer Edge.Cuts) (width 0.1))
-  (gr_line (start 111.76 22.86) (end 111.76 121.92) (angle 90) (layer Edge.Cuts) (width 0.1))
-  (gr_line (start 25.4 22.86) (end 111.76 22.86) (angle 90) (layer Edge.Cuts) (width 0.1))
+  (gr_line (start 25.4 121.92) (end 25.4 22.86) (angle 90) (layer Edge.Cuts) (width 0.5))
+  (gr_line (start 111.76 121.92) (end 25.4 121.92) (angle 90) (layer Edge.Cuts) (width 0.5))
+  (gr_line (start 111.76 22.86) (end 111.76 121.92) (angle 90) (layer Edge.Cuts) (width 0.5))
+  (gr_line (start 25.4 22.86) (end 111.76 22.86) (angle 90) (layer Edge.Cuts) (width 0.5))
   (dimension 99.06 (width 0.3) (layer Dwgs.User)
     (gr_text "99.060 mm" (at 21.51 72.39 270) (layer Dwgs.User)
@@
     (arrow2b (pts (xy 111.76 20.32) (xy 110.633496 20.906421)))
   )
-  (gr_text "TDU\nAudio\nTechnology\nResearch\nClub" (at 80.01 92.71) (layer B.Cu)
+  (gr_text "Audio\nTechnology\nResearch\nClub\nat\nTokyo Denki University" (at 78.105 93.98) (layer B.Cu)
     (effects (font (size 1.5 1.5) (thickness 0.3)) (justify mirror))
   )
@@
     (effects (font (size 1.5 1.5) (thickness 0.3)) (justify mirror))
   )
-  (gr_text GND (at 109.22 72.39 90) (layer B.Cu)
+  (gr_text GND (at 106.045 72.39 90) (layer B.Cu)
     (effects (font (size 1.5 1.5) (thickness 0.3)) (justify mirror))
   )
@@
   (segment (start 74.803 68.784) (end 75.311 68.276) (width 0.5) (layer B.Cu) (net 7))
   (segment (start 75.311 68.276) (end 76.2 68.276) (width 0.5) (layer B.Cu) (net 7))
-  (segment (start 76.835 44.21) (end 76.835 45.623492) (width 1.5) (layer B.Cu) (net 8))
-  (segment (start 76.835 45.623492) (end 77.47 46.258492) (width 1.5) (layer B.Cu) (net 8))
-  (segment (start 77.47 46.258492) (end 77.47 63.146) (width 1.5) (layer B.Cu) (net 8))
+  (segment (start 76.835 44.21) (end 76.849 44.21) (width 1.5) (layer B.Cu) (net 8))
+  (segment (start 76.849 44.21) (end 77.47 44.831) (width 1.5) (layer B.Cu) (net 8))
+  (segment (start 77.47 44.831) (end 77.47 63.146) (width 1.5) (layer B.Cu) (net 8))
   (segment (start 77.47 63.146) (end 76.2 64.416) (width 1.5) (layer B.Cu) (net 8))
   (segment (start 62.23 55.88) (end 62.23 58.08) (width 1.5) (layer B.Cu) (net 9))
@@
   (segment (start 41.91 77.47) (end 44.45 77.47) (width 1.5) (layer B.Cu) (net 15))
   (segment (start 44.45 77.47) (end 48.26 73.66) (width 1.5) (layer B.Cu) (net 15))
-  (segment (start 68.58 64.77) (end 68.58 63.5) (width 1.5) (layer B.Cu) (net 16))
+  (segment (start 66.04 63.5) (end 67.31 63.5) (width 1.5) (layer B.Cu) (net 16))
+  (segment (start 67.31 63.5) (end 68.58 63.5) (width 1.5) (layer B.Cu) (net 16))
+  (segment (start 68.58 64.77) (end 67.31 63.5) (width 1.5) (layer B.Cu) (net 16))
   (segment (start 69.85 66.04) (end 68.58 64.77) (width 1.5) (layer B.Cu) (net 16))
   (segment (start 69.85 66.041) (end 69.85 66.04) (width 1.5) (layer B.Cu) (net 16))
   (segment (start 71.12 67.311) (end 73.66 67.311) (width 1.5) (layer B.Cu) (net 16))
   (segment (start 69.85 66.041) (end 71.12 67.311) (width 1.5) (layer B.Cu) (net 16))
-  (segment (start 66.04 63.5) (end 68.58 63.5) (width 1.5) (layer B.Cu) (net 16))
   (segment (start 38.1 69.85) (end 39.37 69.85) (width 1.5) (layer B.Cu) (net 17))
   (segment (start 39.37 69.85) (end 41.91 67.31) (width 1.5) (layer B.Cu) (net 17))
