File: Audio/LME49810/_autosave-LME49810.kicad_pcb (KiCad board)
At the start: 2 copper layers, 86.4 x 99.1 mm, 37 parts, among them P1 CONN_01X01, P2 CONN_01X01, P3 CONN_01X01, P4 CONN_01X01, P5 CONN_01X01, Q1 NPN(TO-3P-BCE), Q2 PNP(TO-3P-BCE), Q3 NPN(TO-220-BCE), U1 LME49810

Commit message: Fixes on component conflict
LME49810 PCB revised
Changed lines of the file:
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@@
     (links 56)
     (no_connects 0)
-    (area 14.860001 17.47 111.860001 121.970001)
+    (area 14.860001 17.47 112.010001 122.170001)
     (thickness 1.6)
-    (drawings 25)
+    (drawings 27)
     (tracks 134)
     (zones 0)
@@
     (trace_min 0.1)
     (segment_width 0.2)
-    (edge_width 0.1)
+    (edge_width 0.5)
     (via_size 1.5)
     (via_drill 0.75)
@@
     )
   )
+  (dimension 16.51 (width 0.3) (layer Dwgs.User)
+    (gr_text "16.510 mm" (at 26.59 80.645 270) (layer Dwgs.User)
+      (effects (font (size 1.5 1.5) (thickness 0.3)))
+    )
+    (feature1 (pts (xy 38.1 88.9) (xy 25.24 88.9)))
+    (feature2 (pts (xy 38.1 72.39) (xy 25.24 72.39)))
+    (crossbar (pts (xy 27.94 72.39) (xy 27.94 88.9)))
+    (arrow1a (pts (xy 27.94 88.9) (xy 27.353579 87.773496)))
+    (arrow1b (pts (xy 27.94 88.9) (xy 28.526421 87.773496)))
+    (arrow2a (pts (xy 27.94 72.39) (xy 27.353579 73.516504)))
+    (arrow2b (pts (xy 27.94 72.39) (xy 28.526421 73.516504)))
+  )
+  (dimension 16.51 (width 0.3) (layer Dwgs.User)
+    (gr_text "16.510 mm" (at 26.59 64.135 270) (layer Dwgs.User)
+      (effects (font (size 1.5 1.5) (thickness 0.3)))
+    )
+    (feature1 (pts (xy 38.1 72.39) (xy 25.24 72.39)))
+    (feature2 (pts (xy 38.1 55.88) (xy 25.24 55.88)))
+    (crossbar (pts (xy 27.94 55.88) (xy 27.94 72.39)))
+    (arrow1a (pts (xy 27.94 72.39) (xy 27.353579 71.263496)))
+    (arrow1b (pts (xy 27.94 72.39) (xy 28.526421 71.263496)))
+    (arrow2a (pts (xy 27.94 55.88) (xy 27.353579 57.006504)))
+    (arrow2b (pts (xy 27.94 55.88) (xy 28.526421 57.006504)))
+  )
   (gr_text "LME49810 Power Amplifier PCB\nDesigned by T.Hashizume\nDec.2015" (at 82.55 115.57) (layer B.Cu)
     (effects (font (size 1.5 1.5) (thickness 0.3)) (justify mirror))
@@
     (effects (font (size 1.5 1.5) (thickness 0.3)) (justify mirror))
   )
-  (gr_line (start 25.4 121.92) (end 25.4 22.86) (angle 90) (layer Edge.Cuts) (width 0.1))
-  (gr_line (start 111.76 121.92) (end 25.4 121.92) (angle 90) (layer Edge.Cuts) (width 0.1))
-  (gr_line (start 111.76 22.86) (end 111.76 121.92) (angle 90) (layer Edge.Cuts) (width 0.1))
-  (gr_line (start 25.4 22.86) (end 111.76 22.86) (angle 90) (layer Edge.Cuts) (width 0.1))
+  (gr_line (start 25.4 121.92) (end 25.4 22.86) (angle 90) (layer Edge.Cuts) (width 0.5))
+  (gr_line (start 111.76 121.92) (end 25.4 121.92) (angle 90) (layer Edge.Cuts) (width 0.5))
+  (gr_line (start 111.76 22.86) (end 111.76 121.92) (angle 90) (layer Edge.Cuts) (width 0.5))
+  (gr_line (start 25.4 22.86) (end 111.76 22.86) (angle 90) (layer Edge.Cuts) (width 0.5))
   (dimension 99.06 (width 0.3) (layer Dwgs.User)
     (gr_text "99.060 mm" (at 21.51 72.39 270) (layer Dwgs.User)
@@
   (segment (start 74.803 68.784) (end 75.311 68.276) (width 0.5) (layer B.Cu) (net 7))
   (segment (start 75.311 68.276) (end 76.2 68.276) (width 0.5) (layer B.Cu) (net 7))
-  (segment (start 76.835 44.21) (end 76.835 45.623492) (width 1.5) (layer B.Cu) (net 8))
-  (segment (start 76.835 45.623492) (end 77.47 46.258492) (width 1.5) (layer B.Cu) (net 8))
-  (segment (start 77.47 46.258492) (end 77.47 63.146) (width 1.5) (layer B.Cu) (net 8))
+  (segment (start 76.835 44.21) (end 76.849 44.21) (width 1.5) (layer B.Cu) (net 8))
+  (segment (start 76.849 44.21) (end 77.47 44.831) (width 1.5) (layer B.Cu) (net 8))
+  (segment (start 77.47 44.831) (end 77.47 63.146) (width 1.5) (layer B.Cu) (net 8))
   (segment (start 77.47 63.146) (end 76.2 64.416) (width 1.5) (layer B.Cu) (net 8))
   (segment (start 62.23 55.88) (end 62.23 58.08) (width 1.5) (layer B.Cu) (net 9))
