File: Audio/Power_rev.1B/Power.sch (KiCad schematic (older format))
At the start: 38 parts, among them P1 CONN_01X02, P2 CONN_01X02, P3 CONN_01X02, P4 CONN_01X02, Q1 NPN(TO-220-BCE), Q2 PNP(TO-220-BCE), Q3 NPN(TO-220-BCE), Q4 PNP(TO-220-BCE)

Commit message: Further revision
More fixes
Parts:
- C1, C13, C14, C2: footprint Capacitors_ThroughHole:C_Radial_D10_L20_P5-7.5 -> Capacitors_ThroughHole:C_Radial_D10_L20_P7.5
- C10, C9: footprint Capacitors_ThroughHole:C_Radial_D10_L20_P2.5-5 -> Capacitors_ThroughHole:C_Radial_D10_L20_P5
- C11, C12, C3, C4, C5, C6, C7, C8: footprint Capacitors_ThroughHole:C_Disc_D12_P7.75 -> Capacitors_ThroughHole:C_Rect_L13_W4_P10
- D1, D2: symbol DIODE -> DIODE-RESCUE-Power
Changed lines of the file:
@@
 LIBS:Zilog
 LIBS:lme49810
+LIBS:Power-cache
 EELAYER 25 0
 EELAYER END
@@
 F 0 "C1" H 3575 2950 50  0000 L CNN
 F 1 "820uF,100V" H 3575 2750 50  0000 L CNN
-F 2 "Capacitors_ThroughHole:C_Radial_D10_L20_P5-7.5" H 3588 2700 30  0001 C CNN
+F 2 "Capacitors_ThroughHole:C_Radial_D10_L20_P7.5" H 3588 2700 30  0001 C CNN
 F 3 "" H 3550 2850 60  0000 C CNN
 	1    3550 2850
@@
 F 0 "C11" H 6525 2950 50  0000 L CNN
 F 1 "0.1uF,60V+" H 6525 2750 50  0000 L CNN
-F 2 "Capacitors_ThroughHole:C_Disc_D12_P7.75" H 6538 2700 30  0001 C CNN
+F 2 "Capacitors_ThroughHole:C_Rect_L13_W4_P10" H 6538 2700 30  0001 C CNN
 F 3 "" H 6500 2850 60  0000 C CNN
 	1    6500 2850
@@
 F 0 "C13" H 6875 2950 50  0000 L CNN
 F 1 "470uF,200V" H 6875 2750 50  0000 L CNN
-F 2 "Capacitors_ThroughHole:C_Radial_D10_L20_P5-7.5" H 6888 2700 30  0001 C CNN
+F 2 "Capacitors_ThroughHole:C_Radial_D10_L20_P7.5" H 6888 2700 30  0001 C CNN
 F 3 "" H 6850 2850 60  0000 C CNN
 	1    6850 2850
@@
 F 0 "C7" H 5325 2950 50  0000 L CNN
 F 1 "0.1uF,60V+" H 5325 2750 50  0000 L CNN
-F 2 "Capacitors_ThroughHole:C_Disc_D12_P7.75" H 5338 2700 30  0001 C CNN
+F 2 "Capacitors_ThroughHole:C_Rect_L13_W4_P10" H 5338 2700 30  0001 C CNN
 F 3 "" H 5300 2850 60  0000 C CNN
 	1    5300 2850
@@
 $EndComp
 $Comp
-L DIODE D2
+L DIODE-RESCUE-Power D2
 U 1 1 5656CECE
 P 4850 4800
@@
 $EndComp
 $Comp
-L DIODE D1
+L DIODE-RESCUE-Power D1
 U 1 1 5656CE36
 P 4850 1400
@@
 F 0 "C3" H 3875 2950 50  0000 L CNN
 F 1 "0.1uF,125V" H 3875 2750 50  0000 L CNN
-F 2 "Capacitors_ThroughHole:C_Disc_D12_P7.75" H 3888 2700 30  0001 C CNN
+F 2 "Capacitors_ThroughHole:C_Rect_L13_W4_P10" H 3888 2700 30  0001 C CNN
 F 3 "" H 3850 2850 60  0000 C CNN
 	1    3850 2850
@@
 F 0 "C9" H 5525 2950 50  0000 L CNN
 F 1 "22uF,60V+" H 5525 2750 50  0000 L CNN
-F 2 "Capacitors_ThroughHole:C_Radial_D10_L20_P2.5-5" H 5538 2700 30  0001 C CNN
+F 2 "Capacitors_ThroughHole:C_Radial_D10_L20_P5" H 5538 2700 30  0001 C CNN
 F 3 "" H 5500 2850 60  0000 C CNN
 	1    5500 2850
@@
 F 0 "C5" H 4625 2950 50  0000 L CNN
 F 1 "0.47uF,125V" H 4625 2750 50  0000 L CNN
-F 2 "Capacitors_ThroughHole:C_Disc_D12_P7.75" H 4638 2700 30  0001 C CNN
+F 2 "Capacitors_ThroughHole:C_Rect_L13_W4_P10" H 4638 2700 30  0001 C CNN
 F 3 "" H 4600 2850 60  0000 C CNN
 	1    4600 2850
@@
 F 0 "C2" H 3575 3450 50  0000 L CNN
 F 1 "820uF,100V" H 3575 3250 50  0000 L CNN
-F 2 "Capacitors_ThroughHole:C_Radial_D10_L20_P5-7.5" H 3588 3200 30  0001 C CNN
+F 2 "Capacitors_ThroughHole:C_Radial_D10_L20_P7.5" H 3588 3200 30  0001 C CNN
 F 3 "" H 3550 3350 60  0000 C CNN
 	1    3550 3350
@@
 F 0 "C12" H 6525 3450 50  0000 L CNN
 F 1 "0.1uF,60V+" H 6525 3250 50  0000 L CNN
-F 2 "Capacitors_ThroughHole:C_Disc_D12_P7.75" H 6538 3200 30  0001 C CNN
+F 2 "Capacitors_ThroughHole:C_Rect_L13_W4_P10" H 6538 3200 30  0001 C CNN
 F 3 "" H 6500 3350 60  0000 C CNN
 	1    6500 3350
@@
 F 0 "C14" H 6875 3450 50  0000 L CNN
 F 1 "470uF,200V" H 6875 3250 50  0000 L CNN
-F 2 "Capacitors_ThroughHole:C_Radial_D10_L20_P5-7.5" H 6888 3200 30  0001 C CNN
+F 2 "Capacitors_ThroughHole:C_Radial_D10_L20_P7.5" H 6888 3200 30  0001 C CNN
 F 3 "" H 6850 3350 60  0000 C CNN
 	1    6850 3350
@@
 F 0 "C8" H 5325 3450 50  0000 L CNN
 F 1 "0.1uF,60V+" H 5325 3250 50  0000 L CNN
-F 2 "Capacitors_ThroughHole:C_Disc_D12_P7.75" H 5338 3200 30  0001 C CNN
+F 2 "Capacitors_ThroughHole:C_Rect_L13_W4_P10" H 5338 3200 30  0001 C CNN
 F 3 "" H 5300 3350 60  0000 C CNN
 	1    5300 3350
@@
 F 0 "C4" H 3875 3450 50  0000 L CNN
 F 1 "0.1uF,125V" H 3875 3250 50  0000 L CNN
-F 2 "Capacitors_ThroughHole:C_Disc_D12_P7.75" H 3888 3200 30  0001 C CNN
+F 2 "Capacitors_ThroughHole:C_Rect_L13_W4_P10" H 3888 3200 30  0001 C CNN
 F 3 "" H 3850 3350 60  0000 C CNN
 	1    3850 3350
@@
 F 0 "C10" H 5525 3450 50  0000 L CNN
 F 1 "22uF,60V+" H 5525 3250 50  0000 L CNN
-F 2 "Capacitors_ThroughHole:C_Radial_D10_L20_P2.5-5" H 5538 3200 30  0001 C CNN
+F 2 "Capacitors_ThroughHole:C_Radial_D10_L20_P5" H 5538 3200 30  0001 C CNN
 F 3 "" H 5500 3350 60  0000 C CNN
 	1    5500 3350
@@
 F 0 "C6" H 4625 3450 50  0000 L CNN
 F 1 "0.47uF,125V" H 4625 3250 50  0000 L CNN
-F 2 "Capacitors_ThroughHole:C_Disc_D12_P7.75" H 4638 3200 30  0001 C CNN
+F 2 "Capacitors_ThroughHole:C_Rect_L13_W4_P10" H 4638 3200 30  0001 C CNN
 F 3 "" H 4600 3350 60  0000 C CNN
 	1    4600 3350

Commit message: Fixes
More fixes done
Parts:
- removed P1, P2, P3, P4: CONN_01X02, Connect:PINHEAD1-2, symbol CONN_2
- C1, C13, C14, C2: footprint Capacitors_ThroughHole:C_Radial_D10_L20_P7.5 -> Capacitors_ThroughHole:C_Radial_D18_L36_P7.5
- C11, C12, C3, C4, C5, C6, C7, C8: footprint Capacitors_ThroughHole:C_Rect_L13_W4_P10 -> Capacitors_ThroughHole:C_Rect_L18_W6_H12_P15
Connections:
- net GND renamed COM
- net VCC renamed Vcc
- net VEE renamed Vee
Changed lines of the file:
@@
 $EndDescr
-$Comp
-L GND-RESCUE-Power #PWR01
-U 1 1 5656626C
-P 3100 6500
-F 0 "#PWR01" H 3100 6250 50  0001 C CNN
-F 1 "GND" H 3100 6350 50  0000 C CNN
-F 2 "" H 3100 6500 60  0000 C CNN
-F 3 "" H 3100 6500 60  0000 C CNN
-	1    3100 6500
-	1    0    0    -1
-$EndComp
 $Comp
 L CP-RESCUE-Power C1
@@
 F 0 "C1" H 3575 2950 50  0000 L CNN
 F 1 "820uF,100V" H 3575 2750 50  0000 L CNN
-F 2 "Capacitors_ThroughHole:C_Radial_D10_L20_P7.5" H 3588 2700 30  0001 C CNN
+F 2 "Capacitors_ThroughHole:C_Radial_D18_L36_P7.5" H 3588 2700 30  0001 C CNN
 F 3 "" H 3550 2850 60  0000 C CNN
 	1    3550 2850
@@
 Text GLabel 3100 3100 0    60   Input ~ 0
 COM
-Text GLabel 2950 6400 0    60   Output ~ 0
+Text GLabel 3500 6400 2    60   Output ~ 0
 COM
 $Comp
@@
 	0    1    1    0
 $EndComp
-Text GLabel 7550 1700 2    60   Output ~ 0
-VCC
-Text GLabel 7550 4500 2    60   Output ~ 0
-VEE
 $Comp
 L R-RESCUE-Power R9
@@
 F 0 "C11" H 6525 2950 50  0000 L CNN
 F 1 "0.1uF,60V+" H 6525 2750 50  0000 L CNN
-F 2 "Capacitors_ThroughHole:C_Rect_L13_W4_P10" H 6538 2700 30  0001 C CNN
+F 2 "Capacitors_ThroughHole:C_Rect_L18_W6_H12_P15" H 6538 2700 30  0001 C CNN
 F 3 "" H 6500 2850 60  0000 C CNN
 	1    6500 2850
@@
 F 0 "C13" H 6875 2950 50  0000 L CNN
 F 1 "470uF,200V" H 6875 2750 50  0000 L CNN
-F 2 "Capacitors_ThroughHole:C_Radial_D10_L20_P7.5" H 6888 2700 30  0001 C CNN
+F 2 "Capacitors_ThroughHole:C_Radial_D18_L36_P7.5" H 6888 2700 30  0001 C CNN
 F 3 "" H 6850 2850 60  0000 C CNN
 	1    6850 2850
@@
 F 0 "C7" H 5325 2950 50  0000 L CNN
 F 1 "0.1uF,60V+" H 5325 2750 50  0000 L CNN
-F 2 "Capacitors_ThroughHole:C_Rect_L13_W4_P10" H 5338 2700 30  0001 C CNN
+F 2 "Capacitors_ThroughHole:C_Rect_L18_W6_H12_P15" H 5338 2700 30  0001 C CNN
 F 3 "" H 5300 2850 60  0000 C CNN
 	1    5300 2850
@@
 Connection ~ 6000 3100
 $Comp
+L PWR_FLAG #FLG01
+U 1 1 565701F7
+P 3350 5850
+F 0 "#FLG01" H 3350 5945 50  0001 C CNN
+F 1 "PWR_FLAG" H 3350 6030 50  0000 C CNN
+F 2 "" H 3350 5850 60  0000 C CNN
+F 3 "" H 3350 5850 60  0000 C CNN
+	1    3350 5850
+	1    0    0    -1
+$EndComp
+Wire Wire Line
+	3350 6250 3350 6400
+$Comp
 L PWR_FLAG #FLG02
-U 1 1 565701F7
-P 3450 5900
-F 0 "#FLG02" H 3450 5995 50  0001 C CNN
-F 1 "PWR_FLAG" H 3450 6080 50  0000 C CNN
-F 2 "" H 3450 5900 60  0000 C CNN
-F 3 "" H 3450 5900 60  0000 C CNN
-	1    3450 5900
-	1    0    0    -1
-$EndComp
-Wire Wire Line
-	3100 6350 3100 6500
+U 1 1 56574BEF
+P 3350 6250
+F 0 "#FLG02" H 3350 6345 50  0001 C CNN
+F 1 "PWR_FLAG" H 3350 6430 50  0000 C CNN
+F 2 "" H 3350 6250 60  0000 C CNN
+F 3 "" H 3350 6250 60  0000 C CNN
+	1    3350 6250
+	1    0    0    -1
+$EndComp
 $Comp
 L PWR_FLAG #FLG03
-U 1 1 56574BEF
-P 3100 6350
-F 0 "#FLG03" H 3100 6445 50  0001 C CNN
-F 1 "PWR_FLAG" H 3100 6530 50  0000 C CNN
-F 2 "" H 3100 6350 60  0000 C CNN
-F 3 "" H 3100 6350 60  0000 C CNN
-	1    3100 6350
-	-1   0    0    -1
-$EndComp
-Wire Wire Line
-	2950 6000 3500 6000
-$Comp
-L PWR_FLAG #FLG04
 U 1 1 56574FEA
-P 3450 6700
-F 0 "#FLG04" H 3450 6795 50  0001 C CNN
-F 1 "PWR_FLAG" H 3450 6880 50  0000 C CNN
-F 2 "" H 3450 6700 60  0000 C CNN
-F 3 "" H 3450 6700 60  0000 C CNN
-	1    3450 6700
-	-1   0    0    -1
-$EndComp
-Wire Wire Line
-	3450 5900 3450 6000
-Connection ~ 3450 6000
-Wire Wire Line
-	3450 6700 3450 6800
-Connection ~ 3450 6800
+P 3350 6650
+F 0 "#FLG03" H 3350 6745 50  0001 C CNN
+F 1 "PWR_FLAG" H 3350 6830 50  0000 C CNN
+F 2 "" H 3350 6650 60  0000 C CNN
+F 3 "" H 3350 6650 60  0000 C CNN
+	1    3350 6650
+	-1   0    0    -1
+$EndComp
 $Comp
 L R-RESCUE-Power R3
@@
 F 0 "C3" H 3875 2950 50  0000 L CNN
 F 1 "0.1uF,125V" H 3875 2750 50  0000 L CNN
-F 2 "Capacitors_ThroughHole:C_Rect_L13_W4_P10" H 3888 2700 30  0001 C CNN
+F 2 "Capacitors_ThroughHole:C_Rect_L18_W6_H12_P15" H 3888 2700 30  0001 C CNN
 F 3 "" H 3850 2850 60  0000 C CNN
 	1    3850 2850
@@
 	-1   0    0    1
 $EndComp
-$Comp
-L CONN_2 P1
-U 1 1 56643F7E
-P 2600 6100
-F 0 "P1" H 2600 6250 50  0000 C CNN
-F 1 "CONN_01X02" V 2700 6100 50  0000 C CNN
-F 2 "Connect:PINHEAD1-2" H 2600 6100 50  0001 C CNN
-F 3 "" H 2600 6100 50  0000 C CNN
-	1    2600 6100
-	-1   0    0    1
-$EndComp
-$Comp
-L CONN_2 P2
-U 1 1 56644019
-P 2600 6700
-F 0 "P2" H 2600 6850 50  0000 C CNN
-F 1 "CONN_01X02" V 2700 6700 50  0000 C CNN
-F 2 "Connect:PINHEAD1-2" H 2600 6700 50  0001 C CNN
-F 3 "" H 2600 6700 50  0000 C CNN
-	1    2600 6700
-	-1   0    0    -1
-$EndComp
-Wire Wire Line
-	2950 6200 3000 6200
-Wire Wire Line
-	3000 6200 3000 6600
-Wire Wire Line
-	3000 6600 2950 6600
-Wire Wire Line
-	2950 6400 3100 6400
-Connection ~ 3000 6400
-Connection ~ 3100 6400
-Wire Wire Line
-	3500 6800 2950 6800
+Wire Wire Line
+	3350 6400 3500 6400
 $Comp
 L CP-RESCUE-Power C9
@@
 F 0 "C5" H 4625 2950 50  0000 L CNN
 F 1 "0.47uF,125V" H 4625 2750 50  0000 L CNN
-F 2 "Capacitors_ThroughHole:C_Rect_L13_W4_P10" H 4638 2700 30  0001 C CNN
+F 2 "Capacitors_ThroughHole:C_Rect_L18_W6_H12_P15" H 4638 2700 30  0001 C CNN
 F 3 "" H 4600 2850 60  0000 C CNN
 	1    4600 2850
@@
 F 0 "C2" H 3575 3450 50  0000 L CNN
 F 1 "820uF,100V" H 3575 3250 50  0000 L CNN
-F 2 "Capacitors_ThroughHole:C_Radial_D10_L20_P7.5" H 3588 3200 30  0001 C CNN
+F 2 "Capacitors_ThroughHole:C_Radial_D18_L36_P7.5" H 3588 3200 30  0001 C CNN
 F 3 "" H 3550 3350 60  0000 C CNN
 	1    3550 3350
@@
 F 0 "C12" H 6525 3450 50  0000 L CNN
 F 1 "0.1uF,60V+" H 6525 3250 50  0000 L CNN
-F 2 "Capacitors_ThroughHole:C_Rect_L13_W4_P10" H 6538 3200 30  0001 C CNN
+F 2 "Capacitors_ThroughHole:C_Rect_L18_W6_H12_P15" H 6538 3200 30  0001 C CNN
 F 3 "" H 6500 3350 60  0000 C CNN
 	1    6500 3350
@@
 F 0 "C14" H 6875 3450 50  0000 L CNN
 F 1 "470uF,200V" H 6875 3250 50  0000 L CNN
-F 2 "Capacitors_ThroughHole:C_Radial_D10_L20_P7.5" H 6888 3200 30  0001 C CNN
+F 2 "Capacitors_ThroughHole:C_Radial_D18_L36_P7.5" H 6888 3200 30  0001 C CNN
 F 3 "" H 6850 3350 60  0000 C CNN
 	1    6850 3350
@@
 F 0 "C8" H 5325 3450 50  0000 L CNN
 F 1 "0.1uF,60V+" H 5325 3250 50  0000 L CNN
-F 2 "Capacitors_ThroughHole:C_Rect_L13_W4_P10" H 5338 3200 30  0001 C CNN
+F 2 "Capacitors_ThroughHole:C_Rect_L18_W6_H12_P15" H 5338 3200 30  0001 C CNN
 F 3 "" H 5300 3350 60  0000 C CNN
 	1    5300 3350
@@
 F 0 "C4" H 3875 3450 50  0000 L CNN
 F 1 "0.1uF,125V" H 3875 3250 50  0000 L CNN
-F 2 "Capacitors_ThroughHole:C_Rect_L13_W4_P10" H 3888 3200 30  0001 C CNN
+F 2 "Capacitors_ThroughHole:C_Rect_L18_W6_H12_P15" H 3888 3200 30  0001 C CNN
 F 3 "" H 3850 3350 60  0000 C CNN
 	1    3850 3350
@@
 F 0 "C6" H 4625 3450 50  0000 L CNN
 F 1 "0.47uF,125V" H 4625 3250 50  0000 L CNN
-F 2 "Capacitors_ThroughHole:C_Rect_L13_W4_P10" H 4638 3200 30  0001 C CNN
+F 2 "Capacitors_ThroughHole:C_Rect_L18_W6_H12_P15" H 4638 3200 30  0001 C CNN
 F 3 "" H 4600 3350 60  0000 C CNN
 	1    4600 3350
@@
 	4400 4800 4400 4500
 Connection ~ 4400 4500
-$Comp
-L GND-RESCUE-Power #PWR05
-U 1 1 5667F445
-P 5400 6500
-F 0 "#PWR05" H 5400 6250 50  0001 C CNN
-F 1 "GND" H 5400 6350 50  0000 C CNN
-F 2 "" H 5400 6500 60  0000 C CNN
-F 3 "" H 5400 6500 60  0000 C CNN
-	1    5400 6500
-	-1   0    0    -1
-$EndComp
-Text GLabel 5550 6400 2    60   Input ~ 0
-COM
-Wire Wire Line
-	5550 6000 5000 6000
-$Comp
-L CONN_2 P3
-U 1 1 5667F466
-P 5900 6100
-F 0 "P3" H 5900 6250 50  0000 C CNN
-F 1 "CONN_01X02" V 6000 6100 50  0000 C CNN
-F 2 "Connect:PINHEAD1-2" H 5900 6100 50  0001 C CNN
-F 3 "" H 5900 6100 50  0000 C CNN
-	1    5900 6100
-	1    0    0    1
-$EndComp
-$Comp
-L CONN_2 P4
-U 1 1 5667F46C
-P 5900 6700
-F 0 "P4" H 5900 6850 50  0000 C CNN
-F 1 "CONN_01X02" V 6000 6700 50  0000 C CNN
-F 2 "Connect:PINHEAD1-2" H 5900 6700 50  0001 C CNN
-F 3 "" H 5900 6700 50  0000 C CNN
-	1    5900 6700
-	1    0    0    -1
-$EndComp
-Wire Wire Line
-	5550 6200 5500 6200
-Wire Wire Line
-	5500 6200 5500 6600
-Wire Wire Line
-	5500 6600 5550 6600
-Wire Wire Line
-	5550 6400 5400 6400
-Connection ~ 5500 6400
-Wire Wire Line
-	5000 6800 5550 6800
-Wire Wire Line
-	5400 6400 5400 6500
-Text GLabel 5000 6000 0    60   Input ~ 0
-VCC
-Text GLabel 5000 6800 0    60   Input ~ 0
-VEE
 Wire Wire Line
 	4400 1400 4650 1400
@@
 Wire Wire Line
 	5050 4800 5300 4800
+Wire Wire Line
+	3350 5850 3350 6000
+Wire Wire Line
+	3350 6000 3500 6000
+Wire Wire Line
+	3350 6650 3350 6800
+Wire Wire Line
+	3350 6800 3500 6800
+Text Label 7550 1700 0    60   ~ 0
+Vcc
+Text Label 7550 4500 0    60   ~ 0
+Vee
 $EndSCHEMATC
