File: Audio/Power_rev.1B/Power.kicad_pcb (KiCad board)
At the start: 2 copper layers, 96.5 x 101.6 mm, 38 parts, among them P1 CONN_01X02, P2 CONN_01X02, P3 CONN_01X02, P4 CONN_01X02, Q1 NPN(TO-220-BCE), Q2 PNP(TO-220-BCE), Q3 NPN(TO-220-BCE), Q4 PNP(TO-220-BCE)

Commit message: Fix
Fixed for ERC cpmpliance.
Routing:
- net VEE: track 91.9 -> 84.7 mm
- net VCC: track 91.9 -> 84.8 mm
- net 63-75V(-): track 77.7 -> 78.4 mm
- net 63-75V(+): track 77.7 -> 78.4 mm
Other:
- net class Default: clearance 0.2 -> 0.6
- net class Large: clearance 0.2 -> 0.6
- rule trace_clearance: 0.2 -> 0.6
Changed lines of the file:
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@@
     (thickness 1.6)
     (drawings 16)
-    (tracks 136)
+    (tracks 144)
     (zones 0)
     (modules 38)
@@
   (setup
     (last_trace_width 1)
-    (trace_clearance 0.2)
+    (trace_clearance 0.6)
     (zone_clearance 0.508)
     (zone_45_only no)
@@
   (net 15 "Net-(R8-Pad1)")
   (net_class Default "This is the default net class."
-    (clearance 0.2)
+    (clearance 0.6)
     (trace_width 1)
     (via_dia 0.6)
@@
   )
   (net_class Large ""
-    (clearance 0.2)
+    (clearance 0.6)
     (trace_width 2)
     (via_dia 0.6)
@@
   (gr_line (start 68.58 22.86) (end 68.58 20.32) (angle 90) (layer Dwgs.User) (width 0.2))
   (gr_line (start 20.32 71.12) (end 116.84 71.12) (angle 90) (layer Dwgs.User) (width 0.2))
+  (segment (start 40.64 38.735) (end 40.005 38.1) (width 2) (layer B.Cu) (net 1))
+  (segment (start 40.005 38.1) (end 26.67 38.1) (width 2) (layer B.Cu) (net 1))
+  (segment (start 42.33926 37.87394) (end 59.14394 37.87394) (width 2) (layer B.Cu) (net 1))
+  (segment (start 59.14394 37.87394) (end 59.53 38.26) (width 2) (layer B.Cu) (net 1))
+  (segment (start 40.64 38.735) (end 41.4782 38.735) (width 2) (layer B.Cu) (net 1))
+  (segment (start 41.4782 38.735) (end 42.33926 37.87394) (width 2) (layer B.Cu) (net 1))
   (segment (start 59.53 38.26) (end 61.91 40.64) (width 2) (layer B.Cu) (net 1))
-  (segment (start 26.67 38.1) (end 33.02 38.1) (width 2) (layer B.Cu) (net 1))
-  (segment (start 33.18 38.26) (end 33.02 38.1) (width 2) (layer B.Cu) (net 1))
-  (segment (start 44.45 38.26) (end 33.18 38.26) (width 2) (layer B.Cu) (net 1))
-  (segment (start 44.45 38.26) (end 59.53 38.26) (width 2) (layer B.Cu) (net 1))
   (segment (start 61.91 40.64) (end 62.23 40.64) (width 2) (layer B.Cu) (net 1))
   (segment (start 59.69 48.26) (end 62.23 45.72) (width 2) (layer B.Cu) (net 1))
@@
   (segment (start 62.23 40.64) (end 62.23 45.72) (width 2) (layer B.Cu) (net 1))
   (segment (start 64.77 48.26) (end 72.39 48.26) (width 2) (layer B.Cu) (net 1))
+  (segment (start 83.82 50.67) (end 83.82 48.26) (width 2) (layer B.Cu) (net 3))
+  (segment (start 89.535 38.22) (end 86.24 38.22) (width 2) (layer B.Cu) (net 3))
+  (segment (start 86.24 38.22) (end 83.82 40.64) (width 2) (layer B.Cu) (net 3))
+  (segment (start 99.48926 37.87394) (end 98.65106 37.87394) (width 2) (layer B.Cu) (net 3))
+  (segment (start 98.65106 37.87394) (end 97.79 38.735) (width 2) (layer B.Cu) (net 3))
+  (segment (start 89.535 38.22) (end 97.275 38.22) (width 2) (layer B.Cu) (net 3))
+  (segment (start 97.275 38.22) (end 97.79 38.735) (width 2) (layer B.Cu) (net 3))
+  (segment (start 99.48926 37.87394) (end 110.26394 37.87394) (width 2) (layer B.Cu) (net 3))
+  (segment (start 110.26394 37.87394) (end 110.49 38.1) (width 2) (layer B.Cu) (net 3))
   (segment (start 86.995 57.15) (end 83.82 53.975) (width 2) (layer B.Cu) (net 3))
   (segment (start 81.28 45.72) (end 83.82 48.26) (width 2) (layer B.Cu) (net 3))
@@
   (segment (start 86.995 60.96) (end 86.995 67.945) (width 2) (layer B.Cu) (net 3))
   (segment (start 83.82 48.26) (end 83.82 53.975) (width 2) (layer B.Cu) (net 3))
-  (segment (start 93.98 38.1) (end 104.14 38.1) (width 2) (layer B.Cu) (net 3))
-  (segment (start 83.82 40.64) (end 86.36 38.1) (width 2) (layer B.Cu) (net 3))
-  (segment (start 86.36 38.1) (end 93.98 38.1) (width 2) (layer B.Cu) (net 3))
-  (segment (start 104.14 38.1) (end 99.06 38.1) (width 2) (layer B.Cu) (net 3))
-  (segment (start 99.06 38.1) (end 104.14 38.1) (width 2) (layer B.Cu) (net 3))
-  (segment (start 110.49 38.1) (end 104.14 38.1) (width 2) (layer B.Cu) (net 3))
   (segment (start 83.82 40.64) (end 83.82 43.18) (width 2) (layer B.Cu) (net 3))
   (segment (start 81.28 38.1) (end 83.82 40.64) (width 2) (layer B.Cu) (net 3))
@@
   (segment (start 77.47 38.1) (end 81.28 38.1) (width 2) (layer B.Cu) (net 3))
   (segment (start 81.28 45.72) (end 72.39 45.72) (width 2) (layer B.Cu) (net 3))
+  (segment (start 40.64 81.915) (end 40.005 81.28) (width 2) (layer B.Cu) (net 4))
+  (segment (start 40.005 81.28) (end 26.67 81.28) (width 2) (layer B.Cu) (net 4))
+  (segment (start 40.64 81.915) (end 41.4782 81.915) (width 2) (layer B.Cu) (net 4))
+  (segment (start 41.4782 81.915) (end 42.33926 81.05394) (width 2) (layer B.Cu) (net 4))
+  (segment (start 42.33926 81.05394) (end 59.46394 81.05394) (width 2) (layer B.Cu) (net 4))
+  (segment (start 59.46394 81.05394) (end 62.23 83.82) (width 2) (layer B.Cu) (net 4))
   (segment (start 64.77 91.44) (end 72.39 91.44) (width 2) (layer B.Cu) (net 4))
   (segment (start 62.23 83.82) (end 62.23 88.9) (width 2) (layer B.Cu) (net 4))
@@
   (segment (start 76.2 99.06) (end 77.47 99.06) (width 2) (layer B.Cu) (net 4))
   (segment (start 59.69 91.44) (end 62.23 88.9) (width 2) (layer B.Cu) (net 4))
-  (segment (start 61.91 83.82) (end 62.23 83.82) (width 2) (layer B.Cu) (net 4))
-  (segment (start 44.45 81.44) (end 59.53 81.44) (width 2) (layer B.Cu) (net 4))
-  (segment (start 44.45 81.44) (end 33.18 81.44) (width 2) (layer B.Cu) (net 4))
-  (segment (start 33.18 81.44) (end 33.02 81.28) (width 2) (layer B.Cu) (net 4))
-  (segment (start 26.67 81.28) (end 33.02 81.28) (width 2) (layer B.Cu) (net 4))
-  (segment (start 59.53 81.44) (end 61.91 83.82) (width 2) (layer B.Cu) (net 4))
   (segment (start 62.23 111.76) (end 53.34 111.76) (width 1) (layer B.Cu) (net 5))
   (segment (start 57.15 111.76) (end 62.23 111.76) (width 1) (layer B.Cu) (net 5))
@@
   (segment (start 64.77 116.84) (end 66.04 115.57) (width 1) (layer B.Cu) (net 5))
   (segment (start 66.04 115.57) (end 67.31 114.3) (width 1) (layer B.Cu) (net 5))
+  (segment (start 83.82 93.77) (end 83.82 91.44) (width 2) (layer B.Cu) (net 6))
+  (segment (start 89.535 81.4) (end 86.24 81.4) (width 2) (layer B.Cu) (net 6))
+  (segment (start 86.24 81.4) (end 83.82 83.82) (width 2) (layer B.Cu) (net 6))
+  (segment (start 99.48926 81.05394) (end 98.65106 81.05394) (width 2) (layer B.Cu) (net 6))
+  (segment (start 98.65106 81.05394) (end 97.79 81.915) (width 2) (layer B.Cu) (net 6))
+  (segment (start 89.535 81.4) (end 97.275 81.4) (width 2) (layer B.Cu) (net 6))
+  (segment (start 97.275 81.4) (end 97.79 81.915) (width 2) (layer B.Cu) (net 6))
+  (segment (start 99.48926 81.05394) (end 110.26394 81.05394) (width 2) (layer B.Cu) (net 6))
+  (segment (start 110.26394 81.05394) (end 110.49 81.28) (width 2) (layer B.Cu) (net 6))
   (segment (start 81.28 88.9) (end 72.39 88.9) (width 2) (layer B.Cu) (net 6))
   (segment (start 77.47 81.28) (end 81.28 81.28) (width 2) (layer B.Cu) (net 6))
@@
   (segment (start 81.28 81.28) (end 83.82 83.82) (width 2) (layer B.Cu) (net 6))
   (segment (start 83.82 83.82) (end 83.82 86.36) (width 2) (layer B.Cu) (net 6))
-  (segment (start 110.49 81.28) (end 104.14 81.28) (width 2) (layer B.Cu) (net 6))
-  (segment (start 99.06 81.28) (end 104.14 81.28) (width 2) (layer B.Cu) (net 6))
-  (segment (start 104.14 81.28) (end 99.06 81.28) (width 2) (layer B.Cu) (net 6))
-  (segment (start 86.36 81.28) (end 93.98 81.28) (width 2) (layer B.Cu) (net 6))
-  (segment (start 83.82 83.82) (end 86.36 81.28) (width 2) (layer B.Cu) (net 6))
-  (segment (start 93.98 81.28) (end 104.14 81.28) (width 2) (layer B.Cu) (net 6))
   (segment (start 83.82 91.44) (end 83.82 97.155) (width 2) (layer B.Cu) (net 6))
   (segment (start 86.995 104.14) (end 86.995 111.125) (width 2) (layer B.Cu) (net 6))

Commit message: further tweaking(1)
Parts:
- moved R8 28.7 mm to (79.4, 76.8), turned to 90 degrees
- moved R5 23.6 mm to (79.4, 38.7), turned to 270 degrees
- moved R2 23.0 mm to (68.6, 76.2), turned to 270 degrees
- moved C12 22.9 mm to (89.5, 79.4)
- moved C3 19.7 mm to (54.6, 29.2), turned to 270 degrees
- moved D4 19.3 mm to (51.4, 97.8)
- moved C5 19.3 mm to (56.5, 47.0), turned to 270 degrees
- moved Q4 19.1 mm to (64.1, 90.2)
- moved R4 19.1 mm to (74.3, 95.2)
- moved RV2 19.1 mm to (74.3, 90.2)
- moved R7 19.1 mm to (84.5, 90.2)
- moved R1 18.0 mm to (68.6, 38.1), turned to 90 degrees
- moved C11 17.9 mm to (89.5, 33.7)
- moved Q2 17.3 mm to (74.3, 74.3)
- moved C4 16.6 mm to (54.0, 74.9), turned to 90 degrees
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Routing:
- net 63-75V(-): track 78.4 -> 47.8 mm
- net 63-75V(+): track 78.4 -> 47.8 mm
- net Net-(C10-Pad2): track 54.5 -> 42.4 mm
- net Net-(C7-Pad1): track 54.5 -> 42.4 mm
- net VCC: track 84.8 -> 77.0 mm
- net VEE: track 84.7 -> 77.0 mm
- net Net-(R7-Pad2): track 7.62 -> 5.08 mm
- net Net-(R6-Pad1): track 7.62 -> 5.08 mm
- net Net-(R5-Pad2): track 4.97 -> 7.14 mm
- net Net-(R8-Pad1): track 4.97 -> 7.14 mm
- net Net-(C5-Pad1): track 34.4 -> 32.5 mm
- net Net-(C6-Pad2): track 34.4 -> 32.5 mm
Other:
- board size 96.5 x 101.6 mm -> 83.8 x 76.2 mm

Commit message: Further revision
More fixes
Parts:
- C1, C13, C14, C2: footprint Capacitors_ThroughHole:C_Radial_D10_L20_P5-7.5 -> Capacitors_ThroughHole:C_Radial_D10_L20_P7.5
- C10, C9: footprint Capacitors_ThroughHole:C_Radial_D10_L20_P2.5-5 -> Capacitors_ThroughHole:C_Radial_D10_L20_P5
- C11, C12, C3, C4, C5, C6, C7, C8: footprint Capacitors_ThroughHole:C_Disc_D12_P7.75 -> Capacitors_ThroughHole:C_Rect_L13_W4_P10
- moved C8 39.9 mm to (11.3, 76.2), turned to 180 degrees
- moved C6 22.7 mm to (63.5, 71.1), turned to 270 degrees
- moved C11 10.2 mm to (88.9, 43.8), turned to 90 degrees
- moved C5 7.43 mm to (63.5, 44.5), turned to 90 degrees
- moved C4 6.96 mm to (57.1, 81.1)
- moved C1 5.46 mm to (46.4, 29.2)
- moved C10 5.39 mm to (36.8, 85.1)
- moved D4 5.23 mm to (50.2, 92.7)
- moved C2 4.49 mm to (42.5, 74.9)
- moved C9 4.22 mm to (43.2, 53.9)
- moved D3 4.07 mm to (57.8, 57.1)
- moved C13 3.69 mm to (99.1, 49.6), turned to 270 degrees
- moved C14 3.69 mm to (99.1, 87.8)
- moved D2 3.42 mm to (73.0, 66.0)
- moved C7 3.31 mm to (52.7, 53.8)
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Routing:
- net COM: track 0.00 -> 55.1 mm
- net VCC: track 77.0 -> 37.3 mm
- net Net-(C10-Pad2): track 42.4 -> 18.0 mm
- net Net-(C6-Pad2): track 32.5 -> 12.6 mm
- net Net-(C7-Pad1): track 42.4 -> 27.5 mm
- net 63-75V(-): track 47.8 -> 35.8 mm
- net 63-75V(+): track 47.8 -> 53.5 mm
- net VEE: track 77.0 -> 75.1 mm
- net Net-(Q3-Pad1): track 10.2 -> 11.8 mm
- net Net-(C5-Pad1): track 32.5 -> 33.5 mm

Commit message: Fixes
More fixes done
Parts:
- removed P1, P2, P3, P4: CONN_01X02, Connect:PINHEAD1-2
- C1, C13, C14, C2: footprint Capacitors_ThroughHole:C_Radial_D10_L20_P7.5 -> Capacitors_ThroughHole:C_Radial_D18_L36_P7.5
- C11, C12, C3, C4, C5, C6, C7, C8: footprint Capacitors_ThroughHole:C_Rect_L13_W4_P10 -> Capacitors_ThroughHole:C_Rect_L18_W6_H12_P15
- moved C5 50.8 mm to (12.7, 42.9)
- moved R1 50.6 mm to (24.1, 15.2)
- moved C3 45.8 mm to (11.4, 31.8)
- moved R5 45.3 mm to (123.2, 50.2)
- moved C8 41.8 mm to (52.7, 81.9), turned to 270 degrees
- moved R9 40.4 mm to (122.6, 27.9)
- moved C11 40.3 mm to (123.2, 65.0), turned to 270 degrees
- moved C13 17.8 mm to (99.1, 31.9)
- moved C1 11.1 mm to (35.6, 31.8)
- moved C7 7.75 mm to (49.5, 46.8)
- moved C10 6.63 mm to (43.2, 87.0)
- moved C2 3.81 mm to (46.4, 74.9)
- moved C4 3.65 mm to (57.1, 77.5)
- moved D4 3.59 mm to (47.6, 95.2)
- moved D1 3.17 mm to (59.7, 31.8)
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Connections:
- net VCC renamed /Vcc
- net VEE renamed /Vee
Routing:
- net /Vee: track 75.1 -> 0.00 mm
- net COM: track 55.1 -> 0.00 mm
- net 63-75V(-): track 35.8 -> 0.00 mm
- net Net-(C5-Pad1): track 33.5 -> 0.00 mm
- net Net-(C7-Pad1): track 27.5 -> 0.00 mm
- net Net-(C10-Pad2): track 18.0 -> 0.00 mm
- net 63-75V(+): track 53.5 -> 39.8 mm
- net Net-(C6-Pad2): track 12.6 -> 0.00 mm
- net /Vcc: track 37.3 -> 24.8 mm
- net Net-(Q3-Pad1): track 11.8 -> 0.00 mm
- net Net-(Q4-Pad1): track 10.2 -> 0.00 mm
- net Net-(R5-Pad2): track 7.14 -> 0.00 mm
- net Net-(R8-Pad1): track 7.14 -> 0.00 mm
- net Net-(R7-Pad2): track 5.08 -> 0.00 mm
- net Net-(R6-Pad1): track 5.08 -> 0.00 mm

Commit message: Fixes on component conflict
LME49810 PCB revised
Parts:
- C12, C7, C8: footprint Capacitors_ThroughHole:C_Rect_L18_W6_H12_P15 -> Capacitors_ThroughHole:C_Rect_L7.5_W6.5_P5
- moved C5 65.8 mm to (78.5, 44.5), turned to 180 degrees
- moved R1 58.7 mm to (78.7, 36.8), turned to 180 degrees
- moved C3 44.5 mm to (55.9, 31.8)
- moved C11 39.7 mm to (101.6, 31.8)
- moved R5 33.3 mm to (92.7, 36.8)
- moved C9 31.3 mm to (68.6, 35.6), turned to 180 degrees
- moved C13 20.3 mm to (119.4, 31.8)
- moved C7 19.8 mm to (68.6, 52.1), turned to 180 degrees
- moved R9 18.5 mm to (108.0, 39.4), turned to 270 degrees
- moved D3 15.9 mm to (73.7, 57.1)
- moved Q3 15.3 mm to (78.7, 53.3)
- moved RV1 14.6 mm to (88.9, 49.5)
- moved Q1 14.6 mm to (88.9, 34.3)
- moved D1 14.0 mm to (73.7, 31.8)
- moved R6 13.4 mm to (97.8, 52.1)
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Routing:
- net Net-(C7-Pad1): track 0.00 -> 34.4 mm
- net /Vcc: track 24.8 -> 59.0 mm
- net Net-(C5-Pad1): track 0.00 -> 32.4 mm
- net 63-75V(+): track 39.8 -> 52.9 mm
- net Net-(Q3-Pad1): track 0.00 -> 11.7 mm
- net Net-(R5-Pad2): track 0.00 -> 4.86 mm
- net Net-(R6-Pad1): track 0.00 -> 4.86 mm
Other:
- board size 83.8 x 76.2 mm -> 104.1 x 76.2 mm
- net class Default: clearance 0.6 -> 0.2; trace_width 1 -> 1.5
- net class Large: clearance 0.6 -> 0.2
- rule trace_clearance: 0.6 -> 0.2
